File: kicad/solar-system-controller.sch (KiCad schematic (older format))
At the start: 15 parts, among them J1 Raspberry_Pi_2_3, J2 Line_In, U1 MCP3008, U2 500 Gain, U3 1000 Gain

Commit message: Working on the schematic.
Parts:
- added U?: DIFF_ADC, Package_DIP:DIP-16_W7.62mm, symbol Analog_ADC:MCP3008
- added U? (x2): DC-DC-5V, Converter_DCDC:Converter_DCDC_muRata_OKI-78SR_Vertical, symbol Converter_DCDC:OKI-78SR-5_1.5-W36-C
- R?: value 190 -> 105
Connections:
- net LINE1_SWITCH_OUT is gone; now on an unnamed net: R?.2
- net SHUNT_ADC_CH7 is gone; now on net SHUNT_ADC_CH6: U?.7 (CH6)
- net PI_3V3: now also U?.15 (Vref), U?.16 (Vdd)
- net PI_5V: no longer J1.2 (5V)
- net PI_GND: now also U?.14 (AGND), U?.9 (DGND); no longer J1.6 (GND)
- net SHUNT_ADC_CH1: now also U?.2 (CH1); no longer U3.1, U?.1 (CH0)
- net SHUNT_ADC_CH2: now also U?.3 (CH2); no longer U?.2 (CH1)
- net SHUNT_ADC_CH3: now also U?.4 (CH3); no longer U?.3 (CH2)
- net SHUNT_ADC_CH4: now also U?.5 (CH4); no longer U?.4 (CH3)
- net SHUNT_ADC_CH5: now also U?.6 (CH5); no longer U?.5 (CH4)
- net SHUNT_ADC_CH6: no longer U?.6 (CH5)
- net DIFF_ADC_PAIR1_HIGH: now reaches J2.2 (Pin_2), R1.1
- net DIFF_ADC_PAIR1_HIGH: now also U?.1 (CH0)
- net DIFF_ADC_PAIR1_LOW: now reaches F1.1, J2.1 (Pin_1)
- net DIFF_ADC_PAIR1_LOW: now also U?.2 (CH1)
- net PI_CE3: now reaches J1.13 (GPIO27)
- net PI_MOSI: now reaches J1.19 (MOSI0/GPIO10)
- net PI_MOSI: now also U?.11 (Din), U?.11 (Din)
- net PI_MISO: now reaches J1.21 (MISO0/GPIO9)
- net PI_MISO: now also U?.12 (Dout), U?.12 (Dout)
- net PI_SCLK: now reaches J1.23 (SCLK0/GPIO11)
- net PI_SCLK: now also U?.13 (CLK), U?.13 (CLK)
- net PI_CE0: now reaches J1.24 (~CE0~/GPIO8)
- net PI_CE0: now also U?.10 (~CS~/SHDN)
- net PI_CE1: now reaches J1.26 (~CE1~/GPIO7)
- net PI_CE1: now also U?.10 (~CS~/SHDN)
- net BUS_SIGNAL_3V3: now reaches SW?.1
- net PI_LINE1_SWITCH: now reaches SW?.4
- net SHUNT_ADC_CH8: no longer names the net of U?.8 (CH7)
- new net BUS_NEG: J1.6 (GND), U?.2 (GND), U?.2 (GND)
- new net BUS_PI_5V: J1.2 (5V), U?.3 (OUT)
- new net BUS_POS: U?.1 (IN), U?.1 (IN)
- new net BUS_UTIL_5V: U?.3 (OUT)
- new net DIFF_ADC_PAIR2_HIGH: U?.3 (CH2)
- new net DIFF_ADC_PAIR2_LOW: U?.4 (CH3)
- new net DIFF_ADC_PAIR3_HIGH: U?.5 (CH4)
- new net DIFF_ADC_PAIR3_LOW: U?.6 (CH5)
- new net DIFF_ADC_PAIR4_HIGH: U?.7 (CH6)
- new net DIFF_ADC_PAIR4_LOW: U?.8 (CH7)
- new net SHUNT_ADC_CH0: U3.1, U?.1 (CH0)
- no-connect marks 0 -> 3
Other:
- moved on the sheet: J2, R?, SW?, U3
Changed lines of the file:
@@
 L Connector:Screw_Terminal_01x02 J2
 U 1 1 60F87626
-P 16350 3250
-F 0 "J2" H 16430 3242 50  0000 L CNN
-F 1 "Line_In" H 16430 3151 50  0000 L CNN
-F 2 "digikey-footprints:Term_Block_1x2_P5.08MM" H 16350 3250 50  0001 C CNN
-F 3 "https://www.we-online.de/katalog/datasheet/691137710002.pdf" H 16350 3250 50  0001 C CNN
-F 4 "https://www.digikey.com/en/products/detail/w%C3%BCrth-elektronik/691137710002/6644051" H 16350 3250 50  0001 C CNN "Part"
-	1    16350 3250
+P 16850 3250
+F 0 "J2" H 16930 3242 50  0000 L CNN
+F 1 "Line_In" H 16930 3151 50  0000 L CNN
+F 2 "digikey-footprints:Term_Block_1x2_P5.08MM" H 16850 3250 50  0001 C CNN
+F 3 "https://www.we-online.de/katalog/datasheet/691137710002.pdf" H 16850 3250 50  0001 C CNN
+F 4 "https://www.digikey.com/en/products/detail/w%C3%BCrth-elektronik/691137710002/6644051" H 16850 3250 50  0001 C CNN "Part"
+	1    16850 3250
 	1    0    0    -1
 $EndComp
@@
 	16100 3200 16100 3250
 Wire Wire Line
-	16100 3250 16150 3250
-Wire Wire Line
 	15950 3200 16100 3200
-Wire Wire Line
-	16150 3350 16100 3350
 Wire Wire Line
 	16100 3350 16100 3400
@@
 L Amplifier_Current:INA181 U3
 U 1 1 60FA462E
-P 15800 4400
-F 0 "U3" H 15950 4550 50  0000 L CNN
-F 1 "1000 Gain" H 15950 4250 50  0000 L CNN
-F 2 "Package_TO_SOT_SMD:SOT-23-" H 15850 4450 50  0001 C CNN
-F 3 "https://www.ti.com/general/docs/suppproductinfo.tsp?distId=10&gotoUrl=https%3A%2F%2Fwww.ti.com%2Flit%2Fgpn%2Fina210" H 15950 4550 50  0001 C CNN
-F 4 "https://www.digikey.com/en/products/detail/texas-instruments/INA212BIDCKT/3675148" H 15800 4400 50  0001 C CNN "Part"
-F 5 "INA212BIDCKT" H 15800 4400 50  0001 C CNN "Number"
-	1    15800 4400
+P 15800 3950
+F 0 "U3" H 15950 4100 50  0000 L CNN
+F 1 "1000 Gain" H 15950 3800 50  0000 L CNN
+F 2 "Package_TO_SOT_SMD:SOT-23-" H 15850 4000 50  0001 C CNN
+F 3 "https://www.ti.com/general/docs/suppproductinfo.tsp?distId=10&gotoUrl=https%3A%2F%2Fwww.ti.com%2Flit%2Fgpn%2Fina210" H 15950 4100 50  0001 C CNN
+F 4 "https://www.digikey.com/en/products/detail/texas-instruments/INA212BIDCKT/3675148" H 15800 3950 50  0001 C CNN "Part"
+F 5 "INA212BIDCKT" H 15800 3950 50  0001 C CNN "Number"
+	1    15800 3950
 	0    1    1    0
 $EndComp
@@
 $EndComp
 Text GLabel 2700 4350 3    50   Input ~ 0
-PI_GND
+BUS_NEG
 Text GLabel 2900 1750 1    50   Input ~ 0
-PI_5V
+BUS_PI_5V
 Text GLabel 3200 1750 1    50   Input ~ 0
 PI_3V3
-Text GLabel 15500 4300 0    50   Input ~ 0
-PI_GND
-Text GLabel 16100 4300 2    50   Input ~ 0
+Text GLabel 15500 3850 0    50   Input ~ 0
+PI_GND
+Text GLabel 16100 3850 2    50   Input ~ 0
 PI_5V
 Wire Wire Line
-	15500 4300 15500 4500
+	15500 3850 15500 4050
 $Comp
 L Analog_ADC:MCP3008 U?
@@
 	8050 4950 8350 4950
 Text GLabel 7550 5150 0    50   Input ~ 0
+SHUNT_ADC_CH0
+Text GLabel 7550 5250 0    50   Input ~ 0
 SHUNT_ADC_CH1
-Text GLabel 7550 5250 0    50   Input ~ 0
+Text GLabel 7550 5350 0    50   Input ~ 0
 SHUNT_ADC_CH2
-Text GLabel 7550 5350 0    50   Input ~ 0
+Text GLabel 7550 5450 0    50   Input ~ 0
 SHUNT_ADC_CH3
-Text GLabel 7550 5450 0    50   Input ~ 0
+Text GLabel 7550 5550 0    50   Input ~ 0
 SHUNT_ADC_CH4
-Text GLabel 7550 5550 0    50   Input ~ 0
+Text GLabel 7550 5650 0    50   Input ~ 0
 SHUNT_ADC_CH5
-Text GLabel 7550 5650 0    50   Input ~ 0
+Text GLabel 7550 5750 0    50   Input ~ 0
 SHUNT_ADC_CH6
-Text GLabel 7550 5750 0    50   Input ~ 0
-SHUNT_ADC_CH7
-Text GLabel 7550 5850 0    50   Input ~ 0
-SHUNT_ADC_CH8
-Text GLabel 15800 4700 3    50   Input ~ 0
-SHUNT_ADC_CH1
-Wire Wire Line
-	15900 3550 15900 4100
-Wire Wire Line
-	15700 3550 15700 4100
+Text GLabel 15800 4250 3    50   Input ~ 0
+SHUNT_ADC_CH0
+Wire Wire Line
+	15900 3550 15900 3650
+Wire Wire Line
+	15700 3550 15700 3650
 Text GLabel 14450 3400 0    50   Input ~ 0
 BUS+
@@
 L Device:R R?
 U 1 1 60FE2F32
-P 14000 1350
-F 0 "R?" H 13930 1304 50  0000 R CNN
-F 1 "190" H 13930 1395 50  0000 R CNN
-F 2 "" V 13930 1350 50  0001 C CNN
-F 3 "~" H 14000 1350 50  0001 C CNN
-	1    14000 1350
-	-1   0    0    1
-$EndComp
-Text GLabel 13850 1200 0    50   Input ~ 0
-LINE1_SWITCH_OUT
+P 13750 1700
+F 0 "R?" V 13550 1750 50  0000 R CNN
+F 1 "105" V 13650 1800 50  0000 R CNN
+F 2 "" V 13680 1700 50  0001 C CNN
+F 3 "~" H 13750 1700 50  0001 C CNN
+	1    13750 1700
+	0    1    1    0
+$EndComp
 Text GLabel 14000 2100 3    50   Input ~ 0
 PI_GND
@@
 $EndComp
 Wire Wire Line
-	13850 1200 14000 1200
-Wire Wire Line
-	14000 1500 14000 1700
-Wire Wire Line
 	14000 1900 14000 2100
 Wire Wire Line
@@
 L Switch:SW_SP3T SW?
 U 1 1 6103112B
-P 11600 3150
-F 0 "SW?" H 11600 3433 50  0000 C CNN
-F 1 "SP3T" H 11600 3342 50  0000 C CNN
-F 2 "custom-footprints:OS103011MS8QP1_SP3T" H 10975 3325 50  0001 C CNN
-F 3 "https://www.ckswitches.com/media/1428/os.pdf" H 10975 3325 50  0001 C CNN
-F 4 "100mA" H 11600 3150 50  0001 C CNN "Current"
-F 5 "https://www.digikey.com/en/products/detail/c-k/OS103011MS8QP1/1981414" H 11600 3150 50  0001 C CNN "Part"
-	1    11600 3150
-	1    0    0    -1
-$EndComp
+P 13250 1700
+F 0 "SW?" H 13250 1983 50  0000 C CNN
+F 1 "SP3T" H 13250 1892 50  0000 C CNN
+F 2 "custom-footprints:OS103011MS8QP1_SP3T" H 12625 1875 50  0001 C CNN
+F 3 "https://www.ckswitches.com/media/1428/os.pdf" H 12625 1875 50  0001 C CNN
+F 4 "100mA" H 13250 1700 50  0001 C CNN "Current"
+F 5 "https://www.digikey.com/en/products/detail/c-k/OS103011MS8QP1/1981414" H 13250 1700 50  0001 C CNN "Part"
+	1    13250 1700
+	-1   0    0    -1
+$EndComp
+Text GLabel 12900 1600 0    50   Input ~ 0
+BUS_SIGNAL_3V3
+Text GLabel 7900 1100 2    50   Input ~ 0
+BUS_PI_5V
+Text GLabel 7900 2100 2    50   Input ~ 0
+BUS_UTIL_5V
+Text GLabel 12900 1800 0    50   Input ~ 0
+PI_LINE1_SWITCH
+Text GLabel 5050 2150 0    50   Input ~ 0
+PI_LINE1_SWITCH
+Wire Wire Line
+	12900 1600 13050 1600
+Wire Wire Line
+	12900 1800 13050 1800
+NoConn ~ 13050 1700
+Wire Wire Line
+	13450 1700 13600 1700
+Wire Wire Line
+	13900 1700 14000 1700
+Text GLabel 16550 3500 3    50   Input ~ 0
+DIFF_ADC_PAIR1_HIGH
+$Comp
+L Analog_ADC:MCP3008 U?
+U 1 1 60FDB10D
+P 11450 5400
+F 0 "U?" H 11100 6000 50  0000 C CNN
+F 1 "DIFF_ADC" H 11100 5900 50  0000 C CNN
+F 2 "Package_DIP:DIP-16_W7.62mm" H 11550 5500 50  0001 C CNN
+F 3 "http://ww1.microchip.com/downloads/en/DeviceDoc/21295d.pdf" H 11550 5500 50  0001 C CNN
+F 4 "https://www.digikey.com/en/products/detail/microchip-technology/MCP3008-I-P/319422" H 11450 5400 50  0001 C CNN "Part"
+	1    11450 5400
+	1    0    0    -1
+$EndComp
+Text GLabel 11350 4900 1    50   Input ~ 0
+PI_3V3
+Wire Wire Line
+	11650 4900 11350 4900
+Wire Wire Line
+	11650 6000 11350 6000
+Text GLabel 11350 6000 3    50   Input ~ 0
+PI_GND
+Text GLabel 10850 5100 0    50   Input ~ 0
+DIFF_ADC_PAIR1_HIGH
+Text GLabel 10850 5200 0    50   Input ~ 0
+DIFF_ADC_PAIR1_LOW
+Text GLabel 10850 5300 0    50   Input ~ 0
+DIFF_ADC_PAIR2_HIGH
+Text GLabel 10850 5400 0    50   Input ~ 0
+DIFF_ADC_PAIR2_LOW
+Text GLabel 10850 5500 0    50   Input ~ 0
+DIFF_ADC_PAIR3_HIGH
+Text GLabel 10850 5600 0    50   Input ~ 0
+DIFF_ADC_PAIR3_LOW
+Text GLabel 10850 5700 0    50   Input ~ 0
+DIFF_ADC_PAIR4_HIGH
+Text GLabel 10850 5800 0    50   Input ~ 0
+DIFF_ADC_PAIR4_LOW
+Text GLabel 16550 3100 1    50   Input ~ 0
+DIFF_ADC_PAIR1_LOW
+Wire Wire Line
+	16100 3350 16550 3350
+Wire Wire Line
+	16100 3250 16550 3250
+Wire Wire Line
+	16550 3500 16550 3350
+Connection ~ 16550 3350
+Wire Wire Line
+	16550 3350 16650 3350
+Wire Wire Line
+	16550 3100 16550 3250
+Connection ~ 16550 3250
+Wire Wire Line
+	16550 3250 16650 3250
+$Comp
+L Converter_DCDC:OKI-78SR-5_1.5-W36-C U?
+U 1 1 6100527D
+P 7600 1100
+F 0 "U?" H 7600 1342 50  0000 C CNN
+F 1 "DC-DC-5V" H 7600 1251 50  0000 C CNN
+F 2 "Converter_DCDC:Converter_DCDC_muRata_OKI-78SR_Vertical" H 7650 850 50  0001 L CIN
+F 3 "https://power.murata.com/data/power/oki-78sr.pdf" H 7600 1100 50  0001 C CNN
+F 4 "https://www.digikey.com/en/products/detail/murata-power-solutions-inc/OKI-78SR-5-1-5-W36-C/2259781" H 7600 1100 50  0001 C CNN "Part"
+F 5 "1.2" H 7600 1100 50  0001 C CNN "Current"
+	1    7600 1100
+	1    0    0    -1
+$EndComp
+$Comp
+L Converter_DCDC:OKI-78SR-5_1.5-W36-C U?
+U 1 1 610063BE
+P 7600 2100
+F 0 "U?" H 7600 2342 50  0000 C CNN
+F 1 "DC-DC-5V" H 7600 2251 50  0000 C CNN
+F 2 "Converter_DCDC:Converter_DCDC_muRata_OKI-78SR_Vertical" H 7650 1850 50  0001 L CIN
+F 3 "https://power.murata.com/data/power/oki-78sr.pdf" H 7600 2100 50  0001 C CNN
+F 4 "https://www.digikey.com/en/products/detail/murata-power-solutions-inc/OKI-78SR-5-1-5-W36-C/2259781" H 7600 2100 50  0001 C CNN "Part"
+F 5 "1.2" H 7600 2100 50  0001 C CNN "Current"
+	1    7600 2100
+	1    0    0    -1
+$EndComp
+Text GLabel 7300 1100 0    50   Input ~ 0
+BUS_POS
+Text GLabel 7600 1400 3    50   Input ~ 0
+BUS_NEG
+Text GLabel 7300 2100 0    50   Input ~ 0
+BUS_POS
+Text GLabel 7600 2400 3    50   Input ~ 0
+BUS_NEG
+NoConn ~ 15350 3000
+Text GLabel 3900 3550 2    50   Input ~ 0
+PI_SCLK
+Text GLabel 8750 5350 2    50   Input ~ 0
+PI_SCLK
+Text GLabel 3900 3350 2    50   Input ~ 0
+PI_MISO
+Text GLabel 8750 5450 2    50   Input ~ 0
+PI_MISO
+Text GLabel 3900 3450 2    50   Input ~ 0
+PI_MOSI
+Text GLabel 8750 5550 2    50   Input ~ 0
+PI_MOSI
+Text GLabel 3900 3250 2    50   Input ~ 0
+PI_CE0
+Text GLabel 3900 3150 2    50   Input ~ 0
+PI_CE1
+Text GLabel 8750 5650 2    50   Input ~ 0
+PI_CE0
+NoConn ~ 7550 5850
+Text GLabel 12050 5300 2    50   Input ~ 0
+PI_SCLK
+Text GLabel 12050 5400 2    50   Input ~ 0
+PI_MISO
+Text GLabel 12050 5500 2    50   Input ~ 0
+PI_MOSI
+Text GLabel 12050 5600 2    50   Input ~ 0
+PI_CE1
+Text GLabel 2300 3750 0    50   Input ~ 0
+PI_CE3
 $EndSCHEMATC

Commit message: Removed random symbol/footprints library and added them to a single project library.
Parts:
- F1: footprint footprints:3557-2 -> custom-footprints:fuse-holder-3557-2
Changed lines of the file:
@@
 F 0 "F1" V 15603 3200 50  0000 C CNN
 F 1 "5" V 15694 3200 50  0000 C CNN
-F 2 "footprints:3557-2" V 15730 3200 50  0001 C CNN
+F 2 "custom-footprints:fuse-holder-3557-2" V 15730 3200 50  0001 C CNN
 F 3 "~" H 15800 3200 50  0001 C CNN
 	1    15800 3200
